File: FREENFET3.sch (EAGLE design)
At the start: 24 parts, among them IC1 WS2811-SOP8, J1 IN, J2 OUT, Q1 NTD5867NLT4G, Q2 NTD5867NLT4G, Q3 NTD5867NLT4G, Q4 MOSFET-NSOT-323, Q5 MOSFET-NSOT-323, Q6 MOSFET-NSOT-323

Commit message: Final layout
Parts:
- Q4, Q5, Q6: value MOSFET-NSOT-323 -> RJU003N03
Changed lines of the file:
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@@
 <part name="J2" library="freetronics-jon" deviceset="M03" device="PTH" value="OUT"/>
 <part name="GND2" library="freetronics" deviceset="GND" device=""/>
-<part name="Q4" library="freetronics-jon" deviceset="MOSFET-N" device="SOT-323"/>
+<part name="Q4" library="freetronics-jon" deviceset="MOSFET-N" device="SOT-323" value="RJU003N03"/>
 <part name="R1" library="freetronics-master-v1" deviceset="RESISTOR" device="0603" value="1K"/>
 <part name="R2" library="freetronics-master-v1" deviceset="RESISTOR" device="0603" value="10K"/>
@@
 <part name="R3" library="freetronics-master-v1" deviceset="RESISTOR" device="0603" value="10K"/>
 <part name="D2" library="freetronics-master-v1.1" deviceset="M01" device="PTH_LARGE" value="DRAIN"/>
-<part name="Q5" library="freetronics-jon" deviceset="MOSFET-N" device="SOT-323"/>
+<part name="Q5" library="freetronics-jon" deviceset="MOSFET-N" device="SOT-323" value="RJU003N03"/>
 <part name="R4" library="freetronics-master-v1" deviceset="RESISTOR" device="0603" value="1K"/>
 <part name="R6" library="freetronics-master-v1" deviceset="RESISTOR" device="0603" value="10K"/>
@@
 <part name="D3" library="freetronics-master-v1.1" deviceset="M01" device="PTH_LARGE" value="DRAIN"/>
 <part name="SOURCE" library="freetronics-master-v1.1" deviceset="M01" device="PTH_LARGE" value="SOURCE"/>
-<part name="Q6" library="freetronics-jon" deviceset="MOSFET-N" device="SOT-323"/>
+<part name="Q6" library="freetronics-jon" deviceset="MOSFET-N" device="SOT-323" value="RJU003N03"/>
 <part name="R8" library="freetronics-master-v1" deviceset="RESISTOR" device="0603" value="1K"/>
 <part name="R9" library="freetronics-master-v1" deviceset="RESISTOR" device="0603" value="10K"/>
